Commit message: rviz node

File: kinova_description/urdf/j2s7s300_custom copy.urdf (robot description, URDF)
Before this commit: robot j2s7s300, 16 links, 15 joints
Links:
- removed link end_effector
- removed link link_1
- removed link link_2
- removed link link_3
- removed link link_4
- removed link link_5
- removed link link_6
- removed link link_7
- removed link link_base
- removed link link_finger_1
- removed link link_finger_2
- removed link link_finger_3
- removed link link_finger_tip_1
- removed link link_finger_tip_2
- removed link link_finger_tip_3
- added link j2s7s300_end_effector; collision box size=0 0 0; visual box size=0 0 0
- added link j2s7s300_link_1, mass 0.7477; collision mesh filename=package://kinova_description/meshes/shoulder.STL; visual mesh filename=package://kinova_description/meshes/ring_big.STL
- added link j2s7s300_link_2, mass 0.8447; collision mesh filename=package://kinova_description/meshes/arm_half_1.STL; visual mesh filename=package://kinova_description/meshes/arm_half_1.STL
- added link j2s7s300_link_3, mass 0.8447; collision mesh filename=package://kinova_description/meshes/arm_half_2.STL; visual mesh filename=package://kinova_description/meshes/arm_half_2.STL
- added link j2s7s300_link_4, mass 0.6763; collision mesh filename=package://kinova_description/meshes/forearm.STL; visual mesh filename=package://kinova_description/meshes/forearm.STL
- added link j2s7s300_link_5, mass 0.463; collision mesh filename=package://kinova_description/meshes/wrist_spherical_1.STL; visual mesh filename=package://kinova_description/meshes/ring_small.STL
- added link j2s7s300_link_6, mass 0.463; collision mesh filename=package://kinova_description/meshes/wrist_spherical_2.STL; visual mesh filename=package://kinova_description/meshes/ring_small.STL
- added link j2s7s300_link_7, mass 0.727; collision mesh filename=package://kinova_description/meshes/hand_3finger.STL; visual mesh filename=package://kinova_description/meshes/hand_3finger.STL
- added link j2s7s300_link_base, mass 0.46784; collision mesh filename=package://kinova_description/meshes/base.STL; visual mesh filename=package://kinova_description/meshes/base.STL
Joints:
- removed joint joint_1
- removed joint joint_2
- removed joint joint_3
- removed joint joint_4
- removed joint joint_5
- removed joint joint_6
- removed joint joint_7
- removed joint joint_base
- removed joint joint_end_effector
- removed joint joint_finger_1
- removed joint joint_finger_2
- removed joint joint_finger_3
- removed joint joint_finger_tip_1
- removed joint joint_finger_tip_2
- removed joint joint_finger_tip_3
- added joint j2s7s300_joint_1: type continuous, parent j2s7s300_link_base, child j2s7s300_link_1, origin xyz=0 0 0.15675 rpy=0 3.14159265359 0, axis 0 0 1, limit lower=-6.28318530718 upper=6.28318530718 effort=2000 velocity=1
- added joint j2s7s300_joint_2: type revolute, parent j2s7s300_link_1, child j2s7s300_link_2, origin xyz=0 0.0016 -0.11875 rpy=-1.57079632679 0 3.14159265359, axis 0 0 1, limit lower=0.523598775598 upper=5.75958653158 effort=2000 velocity=1
- added joint j2s7s300_joint_3: type continuous, parent j2s7s300_link_2, child j2s7s300_link_3, origin xyz=0 -0.205 0 rpy=-1.57079632679 0 0, axis 0 0 1, limit lower=-6.28318530718 upper=6.28318530718 effort=2000 velocity=1
- added joint j2s7s300_joint_4: type revolute, parent j2s7s300_link_3, child j2s7s300_link_4, origin xyz=0 0 -0.205 rpy=1.57079632679 0 3.14159265359, axis 0 0 1, limit lower=0.523598775598 upper=5.75958653158 effort=2000 velocity=1
- added joint j2s7s300_joint_5: type continuous, parent j2s7s300_link_4, child j2s7s300_link_5, origin xyz=0 0.2073 -0.0114 rpy=-1.57079632679 0 3.14159265359, axis 0 0 1, limit lower=-6.28318530718 upper=6.28318530718 effort=2000 velocity=1
- added joint j2s7s300_joint_6: type revolute, parent j2s7s300_link_5, child j2s7s300_link_6, origin xyz=0 0 -0.10375 rpy=1.57079632679 0 3.14159265359, axis 0 0 1, limit lower=0.523598775598 upper=5.75958653158 effort=2000 velocity=1
- added joint j2s7s300_joint_7: type continuous, parent j2s7s300_link_6, child j2s7s300_link_7, origin xyz=0 0.10375 0 rpy=-1.57079632679 0 3.14159265359, axis 0 0 1, limit lower=-6.28318530718 upper=6.28318530718 effort=2000 velocity=1
- added joint j2s7s300_joint_base: type fixed, parent root, child j2s7s300_link_base, origin xyz=0 0 0 rpy=0 0 0, axis 0 0 0, limit lower=0 upper=0 effort=2000 velocity=1
